File: kicad_project/split_kb.kicad_sch (KiCad schematic)
At the start: 122 parts, among them J1 Conn_01x03_Pin, J2 Conn_01x04_Socket, J3 4P4C, SW1 B3S-1002

Commit message: Completed first draft of the PCB
Parts:
- removed D_back_1, D_back_10, D_back_11, D_back_12, D_back_13, D_back_14, D_back_15, D_back_16, D_back_17, D_back_18, D_back_19, D_back_2, D_back_20, D_back_21, D_back_22, D_back_23, D_back_24, D_back_25, D_back_26, D_back_27, D_back_28, D_back_3, D_back_4, D_back_5, D_back_6, D_back_7, D_back_8, D_back_9, D_front_1, D_front_10, D_front_11, D_front_12, D_front_13, D_front_14, D_front_15, D_front_16, D_front_17, D_front_18, D_front_19, D_front_2, D_front_20, D_front_21, D_front_22, D_front_23, D_front_24, D_front_25, D_front_26, D_front_27, D_front_28, D_front_3, D_front_4, D_front_5, D_front_6, D_front_7, D_front_8, D_front_9: BAT42W-V, Diode_SMD:D_SOD-123, symbol Diode:BAT42W-V
- removed J1: Conn_01x03_Pin, Connector_PinHeader_2.54mm:PinHeader_1x03_P2.54mm_Vertical, symbol Connector:Conn_01x03_Pin
- removed SW1: B3S-1002, B3S-1002:SW_B3S-1000_OMR, symbol B3S-1002:B3S-1002
- added D1, D10, D11, D12, D13, D14, D15, D16, D17, D18, D19, D2, D20, D21, D22, D23, D24, D25, D26, D27, D28, D3, D4, D5, D6, D7, D8, D9: 1N5711, Diode_THT:D_DO-35_SOD27_P7.62mm_Horizontal, symbol Diode:1N5711
- added H5: MountingHole, MountingHole:MountingHole_3mm_Pad_Via, symbol Mechanical:MountingHole
- added J1: 4P4C, Connector_RJ:RJ9_Evercom_5301-440xxx_Horizontal, symbol Connector:4P4C
- added J4: Conn_01x04_Pin, Connector_PinHeader_2.54mm:PinHeader_1x04_P2.54mm_Vertical, symbol Connector:Conn_01x04_Pin
- added R0, R1, R2, R3: R, Resistor_THT:R_Axial_DIN0204_L3.6mm_D1.6mm_P5.08mm_Horizontal, symbol Device:R
Connections:
- net EN_JUMP: now also J4.2 (Pin_2)
- net GND: now also J1.1, J4.4 (Pin_4)
- net ROW_0: now also R0.1
- net ROW_1: now also R1.1
- net ROW_2: now also R2.1
- net ROW_3: now also R3.1
- net RST: now also J4.3 (Pin_3)
- net UART_RX: now also J1.3
- net UART_TX: now also J1.2
- net VCC: now also J1.4, J4.1 (Pin_1)
- net at SW_back_8.2, SW_front_8.2: now also D8.2 (A)
- net at SW_back_13.2, SW_front_13.2: now also D13.2 (A)
- net at SW_back_4.2, SW_front_4.2: now also D4.2 (A)
- net at SW_back_3.2, SW_front_3.2: now also D3.2 (A)
- net at SW_back_2.2, SW_front_2.2: now also D2.2 (A)
- net at SW_back_11.2, SW_front_11.2: now also D11.2 (A)
- net at SW_back_18.2, SW_front_18.2: now also D18.2 (A)
- net at SW_back_20.2, SW_front_20.2: now also D20.2 (A)
- net at SW_back_14.2, SW_front_14.2: now also D14.2 (A)
- net at SW_back_17.2, SW_front_17.2: now also D17.2 (A)
- net at SW_back_23.2, SW_front_23.2: now also D23.2 (A)
- net at SW_back_1.2, SW_front_1.2: now also D1.2 (A)
- net at SW_back_5.2, SW_front_5.2: now also D5.2 (A)
- net at SW_back_27.2, SW_front_27.2: now also D27.2 (A)
- net at SW_back_16.2, SW_front_16.2: now also D16.2 (A)
- net at SW_back_24.2, SW_front_24.2: now also D24.2 (A)
- net at SW_back_15.2, SW_front_15.2: now also D15.2 (A)
- net at SW_back_7.2, SW_front_7.2: now also D7.2 (A)
- net at SW_back_25.2, SW_front_25.2: now also D25.2 (A)
- net at SW_back_9.2, SW_front_9.2: now also D9.2 (A)
- net at SW_back_6.2, SW_front_6.2: now also D6.2 (A)
- net at SW_back_10.2, SW_front_10.2: now also D10.2 (A)
- net at SW_back_12.2, SW_front_12.2: now also D12.2 (A)
- net at SW_back_22.2, SW_front_22.2: now also D22.2 (A)
- net at SW_back_19.2, SW_front_19.2: now also D19.2 (A)
- net at SW_back_26.2, SW_front_26.2: now also D26.2 (A)
- net at SW_back_28.2, SW_front_28.2: now also D28.2 (A)
- net at SW_back_21.2, SW_front_21.2: now also D21.2 (A)
- new net: D1.1 (K), D2.1 (K), D3.1 (K), D4.1 (K), D5.1 (K), D6.1 (K), D7.1 (K), R0.2
- new net: D22.1 (K), D23.1 (K), D24.1 (K), D25.1 (K), D26.1 (K), D27.1 (K), D28.1 (K), R3.2
- new net: D10.1 (K), D11.1 (K), D12.1 (K), D13.1 (K), D14.1 (K), D8.1 (K), D9.1 (K), R1.2
- new net: D15.1 (K), D16.1 (K), D17.1 (K), D18.1 (K), D19.1 (K), D20.1 (K), D21.1 (K), R2.2
Other:
- note added: "And just in case, UART is available on those pins"
- note added: "NOTE: AtMel controller do provide a pullup resistor, but not a pulldown (makes sense actually). This imply measurement is done using inverted logic: ROWs are kept at HIGH. Reading ROW is set LOW. The COL connected to a pressed switch will be forced low."
- note added: "Please mount only one..."
- note removed: "The board mounting the microcontroller to not embed a reset button"
- title: (none) -> Split keyboard PCB
- moved on the sheet: J2, J3, U_front1

Commit message: Grounded EN pin, moved a mounting hole
Connections:
- net GND: now also J4.1 (Pin_1)
- net VCC: no longer J4.1 (Pin_1)
Changed lines of the file:
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@@
+	)
+	(symbol
+		(lib_id "power:GND")
+		(at 50.8 127 180)
+		(unit 1)
+		(exclude_from_sim no)
+		(in_bom yes)
+		(on_board yes)
+		(dnp no)
+		(fields_autoplaced yes)
+		(property "Reference" "#PWR011"
+			(at 50.8 120.65 0)
+			(effects
+				(font
+					(size 1.27 1.27)
+				)
+				(hide yes)
+			)
+		)
+		(property "Value" "GND"
+			(at 50.8 121.92 0)
+			(effects
+				(font
+					(size 1.27 1.27)
+				)
+			)
+		)
+		(property "Footprint" ""
+			(at 50.8 127 0)
+			(effects
+				(font
+					(size 1.27 1.27)
+				)
+				(hide yes)
+			)
+		)
+		(property "Datasheet" ""
+			(at 50.8 127 0)
+			(effects
+				(font
+					(size 1.27 1.27)
+				)
+				(hide yes)
+			)
+		)
+		(property "Description" "Power symbol creates a global label with name \"GND\" , ground"
+			(at 50.8 127 0)
+			(effects
+				(font
+					(size 1.27 1.27)
+				)
+				(hide yes)
+			)
+		)
+		(pin "1"
+		)
+		(instances
+			(project "split_kb"
+				(path "/2d97243e-317c-45d7-bfdf-f717437416be"
+					(reference "#PWR011")
+					(unit 1)
+				)
+			)
+		)
 	)
 	(symbol
@@
 					(unit 1)
 				)
-			)
-		)
-	)
-	(symbol
-		(lib_id "power:VCC")
-		(at 50.8 127 0)
-		(unit 1)
-		(exclude_from_sim no)
-		(in_bom yes)
-		(on_board yes)
-		(dnp no)
-		(fields_autoplaced yes)
-		(property "Reference" "#PWR011"
-			(at 50.8 130.81 0)
-			(effects
-				(font
-					(size 1.27 1.27)
-				)
-				(hide yes)
-			)
-		)
-		(property "Value" "VCC"
-			(at 50.8 121.92 0)
-			(effects
-				(font
-					(size 1.27 1.27)
-				)
-			)
-		)
-		(property "Footprint" ""
-			(at 50.8 127 0)
-			(effects
-				(font
-					(size 1.27 1.27)
-				)
-				(hide yes)
-			)
-		)
-		(property "Datasheet" ""
-			(at 50.8 127 0)
-			(effects
-				(font
-					(size 1.27 1.27)
-				)
-				(hide yes)
-			)
-		)
-		(property "Description" "Power symbol creates a global label with name \"VCC\""
-			(at 50.8 127 0)
-			(effects
-				(font
-					(size 1.27 1.27)
-				)
-				(hide yes)
-			)
-		)
-		(pin "1"
-		)
-		(instances
-			(project "split_kb"
-				(path "/2d97243e-317c-45d7-bfdf-f717437416be"
-					(reference "#PWR011")
-					(unit 1)
-				)
